File: OMAPProc_Rev2.brd (EAGLE design)
At the start: 12 parts

Commit message: Moved some stuff around.
Parts:
- removed SHIFT2: TXS0108E, user:PW_R-PDSO-G20
- moved C32 40.3 mm to (38.1, 1.32)
- moved C30 40.3 mm to (6.25, 1.40)
- moved C31 40.3 mm to (3.76, 1.37)
- moved CAM1 40.3 mm to (9.55, 10.4)
- moved JP11 40.3 mm to (5.03, 17.2)
- moved R18 40.3 mm to (39.3, 1.32)
- moved R19 40.3 mm to (10.8, 18.6)
- moved R20 40.3 mm to (12.6, 18.6)
- moved SHIFT1 40.3 mm to (24.2, 15.6)
- moved C33 40.3 mm to (40.5, 1.32)
- moved SOM1 31.8 mm to (65.7, 11.5)
Connections:
- removed net N$10: SHIFT2.20
- removed net N$4: SHIFT2.18
- removed net N$5: SHIFT2.17
- removed net OMAP_SPI4_CS0: SHIFT2.3
- removed net OMAP_SPI4_IRQ: SHIFT2.4
- removed net OMAP_SPI4_SOMI: SHIFT2.1
- net OMAP_1.8V: no longer SHIFT2.10, SHIFT2.2
- net OMAP_3.3V: no longer SHIFT2.19
- net OMAP_GND: no longer SHIFT2.11
Routing:
- net OMAP_SPI4_IRQ: track 33.8 -> 0.00 mm, vias 3 -> 0
- net N$4: track 20.4 -> 0.00 mm, vias 2 -> 0
- net N$5: track 18.6 -> 0.00 mm, vias 2 -> 0
- net N$10: track 16.0 -> 0.00 mm, vias 2 -> 0
- net OMAP_SPI4_SOMI: track 5.31 -> 0.00 mm, vias 1 -> 0
- net OMAP_SPI4_CS0: track 3.09 -> 0.00 mm, vias 1 -> 0
- net OMAP_1.8V: track 84.1 -> 82.2 mm
- net OMAP_GND: track 123.0 -> 122.0 mm
- net OMAP_3.3V: track 43.6 -> 42.7 mm
Other:
- board outline added: 49.8 x 23.2 mm
- board text removed: "GYRO"
- board text removed: "I2C1"
- board text removed: "I2C2"
- board text removed: "LED"
- board text removed: "RADIO"
- board text removed: "WII"
- board text removed: "XL"
