File: OMAPProc_Rev2.sch (EAGLE design)
At the start: 12 parts

Commit message: Moved some stuff around.
Parts:
- removed SHIFT2: TXS0108E, user:TXS0108E
Connections:
- removed net N$10: SHIFT2.B1
- removed net N$4: SHIFT2.B2
- removed net N$5: SHIFT2.B3
- removed net OMAP_SPI4_CS0: SHIFT2.A2
- removed net OMAP_SPI4_IRQ: SHIFT2.A3
- removed net OMAP_SPI4_SOMI: SHIFT2.A1
- net OMAP_1.8V: no longer SHIFT2.OE, SHIFT2.VCCA
- net OMAP_3.3V: no longer SHIFT2.VCCB
- net OMAP_GND: no longer SHIFT2.GND
Changed lines of the file:
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@@
 <part name="C30" library="SparkFun" deviceset="CAP" device="0402-CAP" value="0.1uF"/>
 <part name="C31" library="SparkFun" deviceset="CAP" device="0402-CAP" value="0.1uF"/>
-<part name="SHIFT2" library="user" deviceset="TXS0108E" device=""/>
 <part name="SHIFT1" library="user" deviceset="TXS0108E" device=""/>
 <part name="R18" library="rcl" deviceset="R-US_" device="R0402" value="4.7k"/>
@@
 <instance part="C30" gate="G$1" x="2.54" y="185.42" rot="R90"/>
 <instance part="C31" gate="G$1" x="12.7" y="180.34" rot="R270"/>
-<instance part="SHIFT2" gate="G$1" x="-55.88" y="-40.64"/>
 <instance part="SHIFT1" gate="G$1" x="-35.56" y="-7.62"/>
 <instance part="R18" gate="G$1" x="-66.04" y="25.4" rot="R180"/>
@@
 <junction x="-10.16" y="25.4"/>
 <label x="-116.84" y="12.7" size="1.778" layer="95"/>
-<pinref part="SHIFT2" gate="G$1" pin="GND"/>
 <pinref part="R18" gate="G$1" pin="1"/>
 <pinref part="SHIFT1" gate="G$1" pin="GND"/>
@@
 <label x="-116.84" y="7.62" size="1.778" layer="95"/>
 <pinref part="SHIFT1" gate="G$1" pin="VCCB"/>
-<pinref part="SHIFT2" gate="G$1" pin="VCCB"/>
 <pinref part="C33" gate="G$1" pin="1"/>
 </segment>
@@
 <label x="-116.84" y="10.16" size="1.778" layer="95"/>
 <pinref part="SHIFT1" gate="G$1" pin="VCCA"/>
-<pinref part="SHIFT2" gate="G$1" pin="VCCA"/>
 <pinref part="SHIFT1" gate="G$1" pin="OE"/>
-<pinref part="SHIFT2" gate="G$1" pin="OE"/>
 <pinref part="R18" gate="G$1" pin="2"/>
 <pinref part="C32" gate="G$1" pin="1"/>
@@
 <wire x1="-76.2" y1="-20.32" x2="-93.98" y2="-20.32" width="0.1524" layer="91"/>
 <label x="-116.84" y="-20.32" size="1.778" layer="95"/>
-<pinref part="SHIFT2" gate="G$1" pin="A1"/>
 </segment>
 </net>
@@
 <wire x1="-78.74" y1="-22.86" x2="-93.98" y2="-22.86" width="0.1524" layer="91"/>
 <label x="-116.84" y="-22.86" size="1.778" layer="95"/>
-<pinref part="SHIFT2" gate="G$1" pin="A2"/>
 </segment>
 </net>
@@
 <wire x1="-81.28" y1="-25.4" x2="-93.98" y2="-25.4" width="0.1524" layer="91"/>
 <label x="-116.84" y="-25.4" size="1.778" layer="95"/>
-<pinref part="SHIFT2" gate="G$1" pin="A3"/>
 </segment>
 </net>
@@
 <wire x1="-40.64" y1="-35.56" x2="-12.7" y2="-35.56" width="0.1524" layer="91"/>
 <wire x1="-12.7" y1="-35.56" x2="-12.7" y2="-22.86" width="0.1524" layer="91"/>
-<pinref part="SHIFT2" gate="G$1" pin="B2"/>
 </segment>
 </net>
@@
 <wire x1="-10.16" y1="-38.1" x2="-10.16" y2="-25.4" width="0.1524" layer="91"/>
 <wire x1="-10.16" y1="-25.4" x2="7.62" y2="-25.4" width="0.1524" layer="91"/>
-<pinref part="SHIFT2" gate="G$1" pin="B3"/>
 </segment>
 </net>
@@
 <wire x1="-40.64" y1="-33.02" x2="-15.24" y2="-33.02" width="0.1524" layer="91"/>
 <wire x1="-15.24" y1="-33.02" x2="-15.24" y2="-20.32" width="0.1524" layer="91"/>
-<pinref part="SHIFT2" gate="G$1" pin="B1"/>
-</segment>
-</net>
+</segment>
+</net>
